Commit message: edit joint2 rpy to -1.57, edit limits of joint2

File: urdf/arm_SDH_URDF.urdf (robot description, URDF)
Before this commit: robot arm_SDH_URDF, 8 links, 7 joints
Joints:
- joint joint_2: limit lower=-3.14 upper=0 effort=1 velocity=0.01 -> lower=-1.75 upper=1.75 effort=1 velocity=0.01; origin xyz=0 0 0.2035 rpy=1.5708 0 0 -> xyz=0 0 0.2035 rpy=1.5708 -1.5708 0

Commit message: first commit

File: urdf/arm_SDH_URDF.urdf (robot description, URDF)
Before this commit: robot arm_SDH_URDF, 8 links, 7 joints
Joints:
- joint gripper1_joint: axis 0 0 -1 -> 0 0 1
- joint gripper2_joint: axis 0 0 -1 -> 0 0 1
- joint joint_1: axis 0 0 -1 -> 0 0 1
- joint joint_2: axis 0 0 -1 -> 0 0 1; origin xyz=0 0 0.2035 rpy=1.5708 -1.5708 0 -> xyz=0.0006 0 0.2044 rpy=1.5749 0 0.0064
- joint joint_3: axis 0 0 -1 -> 0 0 1; origin xyz=0.24983 0.0092539 0 rpy=0 0 0.037024 -> xyz=-0.0010 0.2494 0.002 rpy=-0.0042 0 1.5749
- joint joint_4: axis 0 0 -1 -> 0 0 1; origin xyz=0 0 0 rpy=1.5708 0 1.5533 -> xyz=0 0 0.002 rpy=1.5708 0 1.5545
- joint joint_end: origin xyz=0 0 0.255499999999989 rpy=0 0 0 -> xyz=0 0 0.3013 rpy=0 0 0
